File: FeatherWing_dual_TMC2300/FeatherWing_dual_TMC2300.kicad_sch (KiCad schematic)
At the start: 20 parts, among them U1 TMC2300, U2 SRV05-4, U3 TMC2300, U4 SRV05-4

Commit message: fix image size
Parts:
- added JP1: SolderJumper_3_Open, symbol Jumper:SolderJumper_3_Open
Changed lines of the file:
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@@
+	)
+	(symbol
+		(lib_id "Jumper:SolderJumper_3_Open")
+		(at 35.56 105.41 0)
+		(unit 1)
+		(exclude_from_sim yes)
+		(in_bom no)
+		(on_board yes)
+		(dnp no)
+		(fields_autoplaced yes)
+		(property "Reference" "JP1"
+			(at 35.56 99.06 0)
+			(effects
+				(font
+					(size 1.27 1.27)
+				)
+			)
+		)
+		(property "Value" "SolderJumper_3_Open"
+			(at 35.56 101.6 0)
+			(effects
+				(font
+					(size 1.27 1.27)
+				)
+			)
+		)
+		(property "Footprint" ""
+			(at 35.56 105.41 0)
+			(effects
+				(font
+					(size 1.27 1.27)
+				)
+				(hide yes)
+			)
+		)
+		(property "Datasheet" "~"
+			(at 35.56 105.41 0)
+			(effects
+				(font
+					(size 1.27 1.27)
+				)
+				(hide yes)
+			)
+		)
+		(property "Description" "Solder Jumper, 3-pole, open"
+			(at 35.56 105.41 0)
+			(effects
+				(font
+					(size 1.27 1.27)
+				)
+				(hide yes)
+			)
+		)
+		(pin "1"
+		)
+		(pin "3"
+		)
+		(pin "2"
+		)
+		(instances
+			(project ""
+				(path "/f253d4ba-a6e0-485e-b34a-7d8fcbfee4d7"
+					(reference "JP1")
+					(unit 1)
+				)
+			)
+		)
 	)
 	(symbol
